Commit message: robot description error (not finding correct files

File: src/mm_robot_description/urdf/robot_base.urdf.xacro (robot description, xacro)
@@ -1,10 +1,11 @@
 <?xml version="1.0"?>
 <robot xmlns:xacro="http://www.ros.org/wiki/xacro" name="robot_base">
+<xacro:include filename="$(find mm_robot_description)/urdf/robot_essentials.urdf.xacro" />
 <link name="link_name">
     <visual>
         <origin xyz="0 0 0" rpy="1.5707963267949 0 3.14"/>
         <geometry>
-            <!-- <mesh filename="package://mm_robot_description/meshes/robot_base.stl"/> -->
-            <box size="1.0 1.0 1.0" />
+            <mesh filename="package://mm_robot_description/meshes/robot_base.stl"/>
+            <!-- <box size="1.0 1.0 1.0" /> -->
             <!-- <cylinder radius="1.0" length="1.0"/> -->
         </geometry>
@@ -26,7 +27,11 @@
     </inertial> -->
 </link>
-<xacro:arg name="robot_wheel" prefix="front_left"/>
-<xacro:arg name="robot_wheel" prefix="front_right"/>
-<xacro:arg name="robot_wheel" prefix="rear_left"/>
-<xacro:arg name="robot_wheel" prefix="front_right"/>
+<xacro:robot_wheel prefix="front_left"/>
+<xacro:robot_wheel prefix="front_right"/>
+<xacro:robot_wheel prefix="rear_left"/>
+<xacro:robot_wheel prefix="front_right"/>
+<xacro:wheel_joint prefix="front_left" origin="0.220 0.250 0"/>
+<xacro:wheel_joint prefix="front_right" origin="0.220 -0.250 0"/>
+<xacro:wheel_joint prefix="rear_left" origin="-0.220 0.250 0"/>
+<xacro:wheel_joint prefix="rear_right" origin="-0.220 -0.250 0"/>
 </robot>

File: src/mm_robot_description/urdf/robot_essentials.urdf.xacro (robot description, xacro)
@@ -5,7 +5,7 @@
             <visual>
                 <geometry>
-                    <!-- <mesh filename="package://mm_robot_description/meshes/wheel.stl"/> -->
+                    <mesh filename="package://mm_robot_description/meshes/wheel.stl"/>
                     <!-- <box size="1.0 1.0 1.0" /> -->
-                    <cylinder radius="1.0" length="1.0"/>
+                    <!-- <cylinder radius="1.0" length="1.0"/> -->
                 </geometry>
                 <material name="">
@@ -27,3 +27,11 @@
         </link>
     </xacro:macro>
+    <xacro:macro name="wheel_joint" params="prefix origin">
+        <joint name="${prefix}_wheel_joint" type="continuous">
+            <axis xyz="0 1 0"/>
+            <parent link ="base_link"/>
+            <child link ="${prefix}_wheel"/>
+            <origin rpy ="0 0 0" xyz= "${origin}"/>
+        </joint>
+    </xacro:macro>
 </robot>
