Commit message: adding transmissions

File: src/robot_description/urdf/base_robot.urdf.xacro (robot description, xacro)
@@ -5,8 +5,8 @@
   </link>
   <joint name="base_joint" type="fixed">
-      <parent link="base_footprint"/>
-      <child link="base_link"/>
-      <origin xyz="0 0 135.0" rpy="0 0 0"/>
-      <axis xyz="0.0 0.0 0.0"/>
+    <parent link="base_footprint"/>
+    <child link="base_link"/>
+    <origin xyz="0 0 135.0" rpy="0 0 0"/>
+    <axis xyz="0.0 0.0 0.0"/>
   </joint>
   <link name="base_link">
@@ -22,24 +22,38 @@
       </material>
     </visual>
-    <!-- <collision>
+    <collision>
+      <origin
+      xyz="0 0 0"
+      rpy="1.5707963267949 0 3.14" />
       <geometry>
-        <mesh filename="package://pkg_name/meshes/file_name"/>
-        <box size="1.0 1.0 1.0" />
-        <cylinder radius="1.0" length="1.0"/>
+        <mesh filename="package://robot_description/meshes/robot_base.stl" />
       </geometry>
     </collision>
     <inertial>
-      <mass value="0.0"/>
-      <origin xyz="0.0 0.0 0.0" rpy="0.0 0.0 0.0"/>
-      <inertia ixx="0.0" ixy="0.0" ixz="0.0" iyy="0.0" iyz="0.0" izz="0.0"/>
-    </inertial> -->
+      <origin xyz="0.0030946 4.78250032638821E-11 0.053305"
+      rpy="0.0 0.0 0.0"/>
+      <mass value="47.873"/>
+      <inertia ixx="0.0"
+      ixy="0.774276574699151"
+      ixz="-1.03781944357671E-10"
+      iyy="0.00763014265820928"
+      iyz="1.09578155845563E-12"
+      izz="2.1239326987473"/>
+    </inertial>
   </link>
+  <!-- Wheels-->
   <xacro:robot_wheel prefix="front_left"/>
   <xacro:robot_wheel prefix="front_right"/>
   <xacro:robot_wheel prefix="rear_left"/>
   <xacro:robot_wheel prefix="rear_right"/>
+  <!-- Wheel joints-->
   <xacro:wheel_joint prefix="front_left" origin="0.220 0.250 0"/>
   <xacro:wheel_joint prefix="front_right" origin="0.220 -0.250 0"/>
   <xacro:wheel_joint prefix="rear_left" origin="-0.220 0.250 0"/>
   <xacro:wheel_joint prefix="rear_right" origin="-0.220 -0.250 0"/>
+  <!--Wheel transmissions-->
+  <xacro:base_transmission prefix="front_left"/>
+  <xacro:base_transmission prefix="front_right"/>
+  <xacro:base_transmission prefix="rear_left"/>
+  <xacro:base_transmission prefix="rear_right"/>
 </robot>

File: src/robot_description/urdf/robot_essentials.xacro (robot description, xacro)
@@ -1,4 +1,5 @@
 <?xml version="1.0"?>
 <robot xmlns:xacro="http://ros.org/wiki/xacro" name="robot_essentials" >
+  <!--Wheels-->
   <xacro:macro name="robot_wheel" params="prefix">
     <link name="${prefix}_wheel">
@@ -12,9 +13,31 @@
         <material name="">
           <color
-          rgba="0.79216 0.81961 0.93333 1" />
+            rgba="0.79216 0.81961 0.93333 1" />
         </material>
       </visual>
+      <collision>
+        <origin
+          xyz="0 0 0"
+          rpy="1.5707963267949 0 0" />
+        <geometry>
+          <mesh filename="package://robot_description/meshes/wheel.stl" />
+        </geometry>
+      </collision>
+      <inertial>
+        <origin
+          xyz="-4.1867E-18 0.0068085 -1.65658661799998E-18"
+          rpy="0 0 0" />
+        <mass value="2.6578" />
+        <inertia
+          ixx="0.00856502765719703"
+          ixy="1.5074118157338E-19"
+          ixz="-4.78150098725052E-19"
+          iyy="0.013670640432096"
+          iyz="-2.68136447099727E-19"
+          izz="0.00856502765719703" />
+        </inertial>
     </link>
   </xacro:macro>
+  <!--Wheel joints-->
   <xacro:macro name="wheel_joint" params="prefix origin">
     <joint name="${prefix}_wheel_joint" type="continuous">
@@ -25,3 +48,15 @@
     </joint>
   </xacro:macro>
+  <xacro:macro name="base_transmission" params="prefix ">
+    <transmission name="${prefix}_wheel_trans" type="SimpleTransmission">
+      <type>transmission_interface/SimpleTransmission</type>
+      <actuator name="${prefix}_wheel_motor">
+        <hardwareInterface>hardware_interface/VelocityJointInterface</hardwareInterface>
+        <mechanicalReduction>1</mechanicalReduction>
+      </actuator>
+      <joint name="${prefix}_wheel_joint">
+        <hardwareInterface>hardware_interface/VelocityJointInterface</hardwareInterface>
+      </joint>
+    </transmission>
+  </xacro:macro>
 </robot>

Commit message: adding gazebo plugins

File: src/robot_description/urdf/base_robot.urdf.xacro (robot description, xacro)
@@ -2,5 +2,6 @@
 <robot xmlns:xacro="http://www.ros.org/wiki/xacro" name="robot_base">
   <xacro:include filename="$(find robot_description)/urdf/robot_essentials.xacro"/>
-  <link name="base_footprint">
+  <xacro:include filename="$(find robot_description)/urdf/gazebo_essentials_base.xacro"/>
+  <!-- <link name="base_footprint">
   </link>
   <joint name="base_joint" type="fixed">
@@ -9,5 +10,5 @@
     <origin xyz="0 0 135.0" rpy="0 0 0"/>
     <axis xyz="0.0 0.0 0.0"/>
-  </joint>
+  </joint> -->
   <link name="base_link">
     <visual>
@@ -57,3 +58,8 @@
   <xacro:base_transmission prefix="rear_left"/>
   <xacro:base_transmission prefix="rear_right"/>
+  <!--Wheel friction-->
+  <xacro:wheel_friction prefix="front_left"/>
+  <xacro:wheel_friction prefix="front_right"/>
+  <xacro:wheel_friction prefix="rear_left"/>
+  <xacro:wheel_friction prefix="rear_right"/>
 </robot>
