Commit message: robot arm rendrings successful but needs some tweaks

File: src/robot_description/urdf/robot_essentials.xacro (robot description, xacro)
@@ -1,4 +1,5 @@
 <?xml version="1.0"?>
 <robot xmlns:xacro="http://ros.org/wiki/xacro" name="robot_essentials" >
+<!-- ########################### ROBOT BASE ESSENTIALS-->
   <!--Wheels-->
   <xacro:macro name="robot_wheel" params="prefix">
@@ -60,3 +61,12 @@
     </transmission>
   </xacro:macro>
+  <!-- ################################ ROBOT ARM ESSENTIALS #############################-->
+  <xacro:macro name="arm_joint" params="prefix parent child originxyz originrpy">
+    <joint name="${prefix}_joint" type="continuous">
+      <axis xyz="0 1 0"/>
+      <parent link="${parent}"/>
+      <child link="${child}"/>
+      <origin rpy="${originrpy}" xyz="${originxyz}"/>
+    </joint>
+  </xacro:macro>
 </robot>
