Commit message: robot arm kind of working

File: src/robot_description/urdf/robot_arm.urdf.xacro (robot description, xacro)
@@ -2,5 +2,5 @@
 <robot xmlns:xacro="http://www.ros.org/wiki/xacro" name="robot_name">
   <!-- <xacro:include filename="$(find robot_description)/urdf/robot_arm_essentials.xacro" /> -->
-  <!-- <xacro:include filename="$(find robot_description)/urdf/gazebo_essentials_arm.xacro" /> -->
+  <xacro:include filename="$(find robot_description)/urdf/gazebo_essentials_arm.xacro" />
   <xacro:include filename="$(find robot_description)/urdf/robot_essentials.xacro" />
   <link name="base_footprint">
@@ -214,3 +214,9 @@
   <xacro:arm_joint prefix="top_wrist" parent="elbow" child="top_wrist"
     originxyz="0.0 0 0.20994" originrpy="0 0 0"/>
+  <!-- TRANSMISSIONS -->
+  <xacro:arm_transmission prefix="arm_base"/>
+  <xacro:arm_transmission prefix="shoulder"/>
+  <xacro:arm_transmission prefix="bottom_wrist"/>
+  <xacro:arm_transmission prefix="elbow"/>
+  <xacro:arm_transmission prefix="top_wrist"/>
 </robot>

File: src/robot_description/urdf/robot_essentials.xacro (robot description, xacro)
@@ -1,5 +1,5 @@
 <?xml version="1.0"?>
 <robot xmlns:xacro="http://ros.org/wiki/xacro" name="robot_essentials" >
-<!-- ########################### ROBOT BASE ESSENTIALS-->
+<!-- ########################### ROBOT BASE ESSENTIALS ###########################-->
   <!--Wheels-->
   <xacro:macro name="robot_wheel" params="prefix">
@@ -70,3 +70,15 @@
     </joint>
   </xacro:macro>
+  <xacro:macro name="arm_transmission" params="prefix ">
+    <transmission name="${prefix}_trans" type="SimpleTransmission">
+      <type>transmission_interface/SimpleTransmission</type>
+      <actuator name="${prefix}_motor">
+        <hardwareInterface>hardware_interface/PositionJointInterface</hardwareInterface>
+        <mechanicalReduction>1</mechanicalReduction>
+      </actuator>
+      <joint name="${prefix}_joint">
+        <hardwareInterface>hardware_interface/PositionJointInterface</hardwareInterface>
+      </joint>
+    </transmission>
+  </xacro:macro>
 </robot>

Commit message: simulation in both rviz and gazebo working well. Still not sure about how to control the robot in gazebo

File: src/robot_description/urdf/robot_arm.urdf.xacro (robot description, xacro)
@@ -4,5 +4,5 @@
   <xacro:include filename="$(find robot_description)/urdf/gazebo_essentials_arm.xacro" />
   <xacro:include filename="$(find robot_description)/urdf/robot_essentials.xacro" />
-  <link name="base_footprint">
+  <!-- <link name="base_footprint">
   </link>
   <joint name="base_joint" type="fixed">
@@ -11,5 +11,5 @@
     <origin xyz="0 0 135.0" rpy="0 0 0"/>
     <axis xyz="0.0 0.0 0.0"/>
-  </joint>
+  </joint> -->
   <!-- robot arm base-->
   <link name="arm_base">
@@ -205,5 +205,8 @@
     </collision>
   </link>
+  <!-- <link name="world"/> -->
   <!-- JOINTS -->
+  <!-- <xacro:arm_joint prefix="arm_base" parent="world" child="arm_base"
+    originxyz="0.0 0.0 0.1" originrpy="0 0 0"/> -->
   <xacro:arm_joint prefix="shoulder" parent="arm_base" child="bicep"
     originxyz="-0.05166 0.0 0.20271" originrpy="0 0 1.5708"/>
